File: grblPANEL.kicad_sch (KiCad schematic)
At the start: 0 parts

Commit message: Refresh
Other:
- sheet Testing renamed Misc

Commit message: WIP layout
Other:
- note added: "Note: Investigate options for 4 channel TVS arrays; PESD3V3L4BHC PUSB3AB4 PESD4USB3B Also resistor arrays (for display).."
Changed lines of the file:
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@@
     (effects (font (size 4 4) (thickness 1) bold italic) (justify left bottom))
+  )
+  (text "Note:\n\nInvestigate options for 4 channel TVS arrays;\nPESD3V3L4BHC\nPUSB3AB4\nPESD4USB3B\n\nAlso resistor arrays (for display).."
+    (at 20.32 191.77 0)
+    (effects (font (size 1.27 1.27)) (justify left bottom))
   )
   (text "[6] Keypad" (at 104.14 93.98 0)
@@
       (reference "C502") (unit 1) (value "100n") (footprint "Capacitor_SMD:C_0603_1608Metric")
     )
-    (path "/2c60fe6e-45f9-484b-a2a4-9c1dd728d5af/0d441b06-4635-4e09-a06f-945751747df1"
-      (reference "C503") (unit 1) (value "100n") (footprint "Capacitor_SMD:C_0603_1608Metric")
-    )
     (path "/7148135c-915e-4af4-a225-653bce14d471/e03e009e-f3ce-493f-8aab-8ed0c4528f2f"
       (reference "C601") (unit 1) (value "10u") (footprint "Capacitor_SMD:C_1206_3216Metric")
@@
       (reference "D708") (unit 1) (value "D_TVS") (footprint "Diode_SMD:D_SOD-323")
     )
+    (path "/7148135c-915e-4af4-a225-653bce14d471/0d5d4aba-d658-478e-b973-c3bc44c70fa2"
+      (reference "D?") (unit 1) (value "PESD3V3L4UF") (footprint "Package_TO_SOT_SMD:SOT-886")
+    )
     (path "/d3c757f4-85a2-4c64-b768-7bb57e3daca0/099b9606-b5db-4c56-980a-1663a2896b17"
       (reference "J101") (unit 1) (value "Conn_01x02") (footprint "TerminalBlock_Phoenix:TerminalBlock_Phoenix_PT-1,5-2-3.5-H_1x02_P3.50mm_Horizontal")
@@
       (reference "R502") (unit 1) (value "10k") (footprint "Resistor_SMD:R_0603_1608Metric")
     )
+    (path "/2c60fe6e-45f9-484b-a2a4-9c1dd728d5af/274f34a6-a307-48a7-a660-b805c6ca42ad"
+      (reference "R503") (unit 1) (value "0") (footprint "Resistor_SMD:R_0603_1608Metric")
+    )
     (path "/2c60fe6e-45f9-484b-a2a4-9c1dd728d5af/d3b4e76e-bb50-45c5-b9b3-94e0c997b79c"
-      (reference "R503") (unit 1) (value "5R6") (footprint "Resistor_SMD:R_0603_1608Metric")
-    )
-    (path "/2c60fe6e-45f9-484b-a2a4-9c1dd728d5af/274f34a6-a307-48a7-a660-b805c6ca42ad"
-      (reference "R504") (unit 1) (value "0") (footprint "Resistor_SMD:R_0603_1608Metric")
+      (reference "R504") (unit 1) (value "5R6") (footprint "Resistor_SMD:R_0603_1608Metric")
     )
     (path "/2c60fe6e-45f9-484b-a2a4-9c1dd728d5af/262f5b07-e1ac-4703-8dae-32f0325a4b22"
@@
       (reference "R708") (unit 1) (value "200") (footprint "Resistor_SMD:R_0603_1608Metric")
     )
+    (path "/7148135c-915e-4af4-a225-653bce14d471/6cd39ac1-1cc5-4bb8-ab3f-e9fbacf3fe45"
+      (reference "RN?") (unit 1) (value "R_Pack04") (footprint "")
+    )
     (path "/437f2ceb-712b-41a0-9e79-c6c2becba629/ce40af38-6eca-4492-8fde-6e9a33cb1c65"
