File: grblPANEL_display.kicad_sch (KiCad schematic)
At the start: 16 parts, among them J501 ILI9488, Q501 Q_NPN_BCE

Commit message: ERC fixes
Parts:
- renumbered R504 to R501, R501 to R502, R502 to R504, TP506 to TP502, TP507 to TP503, TP502 to TP504, TP503 to TP505, TP504 to TP506, TP505 to TP507
Connections:
- net DISPLAY_CS: no longer J501.13 (SDA), J501.14 (SDO), TP505.1, TP506.1
- new net DISPLAY_SDA: J501.13 (SDA), TP505.1
- new net DISPLAY_SDO: J501.14 (SDO), TP506.1
Changed lines of the file:
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@@
   (junction (at 162.56 119.38) (diameter 0) (color 0 0 0 0)
   )
-  (junction (at 128.27 66.04) (diameter 0) (color 0 0 0 0)
-  )
   (junction (at 120.65 66.04) (diameter 0) (color 0 0 0 0)
   )
@@
   (junction (at 209.55 93.98) (diameter 0) (color 0 0 0 0)
   )
+  (junction (at 182.88 132.08) (diameter 0) (color 0 0 0 0)
+  )
   (junction (at 209.55 91.44) (diameter 0) (color 0 0 0 0)
   )
@@
   (junction (at 144.78 66.04) (diameter 0) (color 0 0 0 0)
   )
-  (junction (at 132.08 66.04) (diameter 0) (color 0 0 0 0)
-  )
   (junction (at 209.55 109.22) (diameter 0) (color 0 0 0 0)
   )
@@
   )
   (junction (at 162.56 132.08) (diameter 0) (color 0 0 0 0)
-  )
-  (junction (at 182.88 132.08) (diameter 0) (color 0 0 0 0)
   )
   (no_connect (at 203.2 73.66))
@@
     (stroke (width 0) (type default) (color 0 0 0 0))
   )
-  (wire (pts (xy 128.27 57.15) (xy 128.27 66.04))
-    (stroke (width 0) (type default) (color 0 0 0 0))
-  )
-  (wire (pts (xy 132.08 60.96) (xy 132.08 66.04))
+  (wire (pts (xy 128.27 57.15) (xy 128.27 71.12))
+    (stroke (width 0) (type default) (color 0 0 0 0))
+  )
+  (wire (pts (xy 132.08 60.96) (xy 132.08 73.66))
     (stroke (width 0) (type default) (color 0 0 0 0))
   )
@@
     (stroke (width 0) (type default) (color 0 0 0 0))
   )
-  (wire (pts (xy 128.27 66.04) (xy 132.08 66.04))
-    (stroke (width 0) (type default) (color 0 0 0 0))
-  )
   (wire (pts (xy 144.78 59.69) (xy 144.78 66.04))
     (stroke (width 0) (type default) (color 0 0 0 0))
@@
     (stroke (width 0) (type default) (color 0 0 0 0))
   )
+  (wire (pts (xy 182.88 132.08) (xy 209.55 132.08))
+    (stroke (width 0) (type default) (color 0 0 0 0))
+  )
   (wire (pts (xy 120.65 90.17) (xy 167.64 90.17))
     (stroke (width 0) (type default) (color 0 0 0 0))
@@
     (stroke (width 0) (type default) (color 0 0 0 0))
   )
-  (wire (pts (xy 120.65 66.04) (xy 128.27 66.04))
-    (stroke (width 0) (type default) (color 0 0 0 0))
-  )
   (polyline (pts (xy 77.47 26.67) (xy 233.68 26.67))
     (stroke (width 0) (type default) (color 0 0 0 0))
@@
     (stroke (width 0) (type default) (color 0 0 0 0))
   )
-  (wire (pts (xy 128.27 66.04) (xy 128.27 71.12))
-    (stroke (width 0) (type default) (color 0 0 0 0))
-  )
   (wire (pts (xy 209.55 119.38) (xy 209.55 132.08))
     (stroke (width 0) (type default) (color 0 0 0 0))
@@
     (stroke (width 0) (type default) (color 0 0 0 0))
   )
-  (wire (pts (xy 132.08 66.04) (xy 144.78 66.04))
+  (wire (pts (xy 120.65 66.04) (xy 144.78 66.04))
     (stroke (width 0) (type default) (color 0 0 0 0))
   )
@@
     (stroke (width 0) (type default) (color 0 0 0 0))
   )
-  (wire (pts (xy 182.88 132.08) (xy 209.55 132.08))
-    (stroke (width 0) (type default) (color 0 0 0 0))
-  )
   (wire (pts (xy 120.65 121.92) (xy 120.65 125.73))
-    (stroke (width 0) (type default) (color 0 0 0 0))
-  )
-  (wire (pts (xy 132.08 66.04) (xy 132.08 73.66))
     (stroke (width 0) (type default) (color 0 0 0 0))
   )
@@
   (symbol (lib_id "Device:R") (at 158.75 68.58 90) (unit 1)
     (in_bom yes) (on_board yes)
-    (property "Reference" "R502" (id 0) (at 163.83 67.31 90))
+    (property "Reference" "R504" (id 0) (at 163.83 67.31 90))
     (property "Value" "0" (id 1) (at 154.94 67.31 90))
     (property "Footprint" "" (id 2) (at 158.75 70.358 90)
@@
   (symbol (lib_id "Connector:TestPoint") (at 124.46 53.34 0) (unit 1)
     (in_bom yes) (on_board yes)
-    (property "Reference" "TP502" (id 0) (at 124.46 48.26 0)
+    (property "Reference" "TP504" (id 0) (at 124.46 48.26 0)
       (effects (font (size 1.27 1.27)) (justify left))
     )
@@
   (symbol (lib_id "Connector:TestPoint") (at 120.65 121.92 0) (unit 1)
     (in_bom yes) (on_board yes)
-    (property "Reference" "TP507" (id 0) (at 119.38 116.84 0)
+    (property "Reference" "TP503" (id 0) (at 119.38 116.84 0)
       (effects (font (size 1.27 1.27)) (justify left))
     )
@@
   (symbol (lib_id "Connector:TestPoint") (at 128.27 57.15 0) (unit 1)
     (in_bom yes) (on_board yes)
-    (property "Reference" "TP503" (id 0) (at 128.27 52.07 0)
+    (property "Reference" "TP505" (id 0) (at 128.27 52.07 0)
       (effects (font (size 1.27 1.27)) (justify left))
     )
@@
   (symbol (lib_id "Connector:TestPoint") (at 132.08 60.96 0) (unit 1)
     (in_bom yes) (on_board yes)
-    (property "Reference" "TP504" (id 0) (at 132.08 55.88 0)
+    (property "Reference" "TP506" (id 0) (at 132.08 55.88 0)
       (effects (font (size 1.27 1.27)) (justify left))
     )
@@
   (symbol (lib_id "Connector:TestPoint") (at 120.65 86.36 0) (unit 1)
     (in_bom yes) (on_board yes)
-    (property "Reference" "TP506" (id 0) (at 119.38 81.28 0)
+    (property "Reference" "TP502" (id 0) (at 119.38 81.28 0)
       (effects (font (size 1.27 1.27)) (justify left))
     )
@@
   (symbol (lib_id "power:+3V3") (at 158.75 38.1 0) (unit 1)
     (in_bom yes) (on_board yes) (fields_autoplaced)
-    (property "Reference" "#PWR0501" (id 0) (at 158.75 41.91 0)
+    (property "Reference" "#PWR0502" (id 0) (at 158.75 41.91 0)
       (effects (font (size 1.27 1.27)) hide)
     )
@@
   (symbol (lib_id "Device:R") (at 144.78 55.88 0) (unit 1)
     (in_bom yes) (on_board yes) (fields_autoplaced)
-    (property "Reference" "R501" (id 0) (at 147.32 54.6099 0)
+    (property "Reference" "R502" (id 0) (at 147.32 54.6099 0)
       (effects (font (size 1.27 1.27)) (justify left))
     )
@@
   (symbol (lib_id "Connector:TestPoint") (at 135.89 64.77 0) (unit 1)
     (in_bom yes) (on_board yes)
-    (property "Reference" "TP505" (id 0) (at 135.89 59.69 0)
+    (property "Reference" "TP507" (id 0) (at 135.89 59.69 0)
       (effects (font (size 1.27 1.27)) (justify left))
     )
@@
   (symbol (lib_id "power:+3V3") (at 144.78 49.53 0) (unit 1)
     (in_bom yes) (on_board yes) (fields_autoplaced)
-    (property "Reference" "#PWR0502" (id 0) (at 144.78 53.34 0)
+    (property "Reference" "#PWR0501" (id 0) (at 144.78 53.34 0)
       (effects (font (size 1.27 1.27)) hide)
     )
@@
   (symbol (lib_id "Device:R") (at 138.43 125.73 90) (unit 1)
     (in_bom yes) (on_board yes)
-    (property "Reference" "R504" (id 0) (at 138.43 120.65 90))
+    (property "Reference" "R501" (id 0) (at 138.43 120.65 90))
     (property "Value" "1k" (id 1) (at 138.43 123.19 90))
     (property "Footprint" "" (id 2) (at 138.43 127.508 90)

Commit message: Refresh
Parts:
- removed Q501: Q_NPN_BCE, symbol Device:Q_NPN_BCE
- added Q501: Q_NPN_BEC - S8050, Package_TO_SOT_SMD:SOT-23, symbol Device:Q_NPN_BEC
- added R505: 1k, Resistor_SMD:R_0603_1608Metric, symbol Device:R
- C501: footprint (none) -> Capacitor_SMD:C_0805_2012Metric
- C502, C503: footprint (none) -> Capacitor_SMD:C_0603_1608Metric
- J501: footprint (none) -> Connector_FFC-FPC:Hirose_FH12-40S-0.5SH_1x40-1MP_P0.50mm_Horizontal
- R501, R502, R504: footprint (none) -> Resistor_SMD:R_0603_1608Metric
- R503: value 100 -> 5R6; footprint (none) -> Resistor_SMD:R_0603_1608Metric
- TP501, TP502, TP503, TP504, TP505, TP506, TP507: footprint (none) -> Connector_Pin:Pin_D1.0mm_L10.0mm
Connections:
- net GND: now also Q501.2 (E), R505.1; no longer J501.17 (DB0), J501.18 (DB1), J501.19 (DB2), J501.20 (DB3), J501.21 (DB4), J501.22 (DB5), J501.23 (DB6), J501.24 (DB7), J501.25 (DB8), J501.26 (DB9), J501.27 (DB10), J501.28 (DB11), J501.29 (DB12), J501.30 (DB13), J501.31 (DB14), J501.32 (DB15)
- net at R501.2: now also Q501.1 (B)
- net at R503.1: now also Q501.3 (C)
- new net: J501.17 (DB0), J501.18 (DB1), J501.19 (DB2), J501.20 (DB3), J501.21 (DB4), J501.22 (DB5), J501.23 (DB6), J501.24 (DB7), J501.25 (DB8), J501.26 (DB9), J501.27 (DB10), J501.28 (DB11), J501.29 (DB12), J501.30 (DB13), J501.31 (DB14), J501.32 (DB15), R505.2
Other:
- note added: "Notes: Display modules ordered here; https://www.aliexpress.com/item/32829704426.html Schematic loosely based on this; http://www.lcdwiki.com/3.5inch_SPI_Module_ILI9488_SKU:MSP3520 Note only 40 pins on bare displays, using 40 pin 0.5mm FPC connector Some descriptions have CLK and DATA/CMD pins swapped? https://electronics.stackexchange.com/questions/613498/what-are-the-bare-minimum-number-of-pins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"
- note added: "max base current 3.3mA max backlight current ~100mA"
- note removed: "max base current 3.3mA max backlight current 100mA check - probably incorrect due to diode voltage drop??"
- note removed: "schematic loosley based on examples here; http://www.lcdwiki.com/3.5inch_SPI_Module_ILI9488_SKU:MSP3520 note only 40 pins on bare boards.. ordered here; https://www.aliexpress.com/item/32829704426.html https://electronics.stackexchange.com/questions/613498/what-are-the-bare-minimum-number-of-pins-needed-to-connect-to-an-ili9488-tft-in Using 40 pin 0.5mm FPC connector WTF is SPI_AO - the command/d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"

Commit message: PCB layout - WIP
Parts:
- TP501, TP502, TP503, TP504, TP505, TP506, TP507: footprint Connector_Pin:Pin_D1.0mm_L10.0mm -> TestPoint:TestPoint_THTPad_D2.0mm_Drill1.0mm
Changed lines of the file:
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@@
     (effects (font (size 1.27 1.27)) (justify left bottom))
   )
-  (text "Notes:\n\nDisplay modules ordered here;\nhttps://www.aliexpress.com/item/32829704426.html\n\nSchematic loosely based on this;\nhttp://www.lcdwiki.com/3.5inch_SPI_Module_ILI9488_SKU:MSP3520\n\nNote only 40 pins on bare displays, using 40 pin 0.5mm FPC connector \n\nSome descriptions have CLK and DATA/CMD pins swapped?\nhttps://electronics.stackexchange.com/questions/613498/what-are-the-bare-minimum-number-of-pins-needed-to-connect-to-an-ili9488-tft-in\nhttps://github.com/Bodmer/TFT_eSPI/issues/968\nhttps://esp32.com/viewtopic.php?t=25917"
+  (text "Notes:\n\nDisplay modules ordered here;\nhttps://www.aliexpress.com/item/32829704426.html\n\nSchematic loosely based on this;\nhttp://www.lcdwiki.com/3.5inch_SPI_Module_ILI9488_SKU:MSP3520\n\nNote only 40 pins on bare displays, using 40 pin 0.5mm FPC connector \n\nSome descriptions have CLK and DATA/CMD pins swapped?\nhttps://electronics.stackexchange.com/questions/613498/what-are-the-bare-minimum-number-of-pins-needed-to-connect-to-an-ili9488-tft-in\nhttps://github.com/Bodmer/TFT_eSPI/issues/968\nhttps://esp32.com/viewtopic.php?t=25917\n\ntodo: finalise FPC connector footprint once ordered (existing KiCad footprint for Hirose FH12)"
     (at 20.32 190.5 0)
     (effects (font (size 1.27 1.27)) (justify left bottom))
@@
       (effects (font (size 1.27 1.27)) (justify left) hide)
     )
-    (property "Footprint" "Connector_Pin:Pin_D1.0mm_L10.0mm" (id 2) (at 129.54 53.34 0)
+    (property "Footprint" "TestPoint:TestPoint_THTPad_D2.0mm_Drill1.0mm" (id 2) (at 129.54 53.34 0)
       (effects (font (size 1.27 1.27)) hide)
     )
@@
       (effects (font (size 1.27 1.27)) (justify left) hide)
     )
-    (property "Footprint" "Connector_Pin:Pin_D1.0mm_L10.0mm" (id 2) (at 125.73 49.53 0)
+    (property "Footprint" "TestPoint:TestPoint_THTPad_D2.0mm_Drill1.0mm" (id 2) (at 125.73 49.53 0)
       (effects (font (size 1.27 1.27)) hide)
     )
@@
       (effects (font (size 1.27 1.27)) (justify left) hide)
     )
-    (property "Footprint" "Connector_Pin:Pin_D1.0mm_L10.0mm" (id 2) (at 125.73 121.92 0)
+    (property "Footprint" "TestPoint:TestPoint_THTPad_D2.0mm_Drill1.0mm" (id 2) (at 125.73 121.92 0)
       (effects (font (size 1.27 1.27)) hide)
     )
@@
       (effects (font (size 1.27 1.27)) (justify left) hide)
     )
-    (property "Footprint" "Connector_Pin:Pin_D1.0mm_L10.0mm" (id 2) (at 133.35 57.15 0)
+    (property "Footprint" "TestPoint:TestPoint_THTPad_D2.0mm_Drill1.0mm" (id 2) (at 133.35 57.15 0)
       (effects (font (size 1.27 1.27)) hide)
     )
@@
       (effects (font (size 1.27 1.27)) (justify left) hide)
     )
-    (property "Footprint" "Connector_Pin:Pin_D1.0mm_L10.0mm" (id 2) (at 137.16 60.96 0)
+    (property "Footprint" "TestPoint:TestPoint_THTPad_D2.0mm_Drill1.0mm" (id 2) (at 137.16 60.96 0)
       (effects (font (size 1.27 1.27)) hide)
     )
@@
       (effects (font (size 1.27 1.27)) (justify left) hide)
     )
-    (property "Footprint" "Connector_Pin:Pin_D1.0mm_L10.0mm" (id 2) (at 125.73 86.36 0)
+    (property "Footprint" "TestPoint:TestPoint_THTPad_D2.0mm_Drill1.0mm" (id 2) (at 125.73 86.36 0)
       (effects (font (size 1.27 1.27)) hide)
     )
@@
       (effects (font (size 1.27 1.27)) (justify left) hide)
     )
-    (property "Footprint" "Connector_Pin:Pin_D1.0mm_L10.0mm" (id 2) (at 140.97 64.77 0)
-      (effects (font (size 1.27 1.27)) hide)
-    )
+    (property "Footprint" "TestPoint:TestPoint_THTPad_D2.0mm_Drill1.0mm" (id 2) (at 140.97 64.77 0)
+      (effects (font (size 1.27 1.27)) hide)
+    )

Commit message: WIP layout
Parts:
- removed C503: 100n, Capacitor_SMD:C_0603_1608Metric, symbol Device:C
- renumbered R504 to R503, R503 to R504
Connections:
- net DIO_GND: now reaches J501.17 (DB0), J501.18 (DB1), J501.19 (DB2), J501.20 (DB3), J501.21 (DB4), J501.22 (DB5), J501.23 (DB6), J501.24 (DB7), J501.25 (DB8), J501.26 (DB9), J501.27 (DB10), J501.28 (DB11), J501.29 (DB12), J501.30 (DB13), J501.31 (DB14), J501.32 (DB15), R505.2
- net BL_K: now reaches J501.34 (K1), J501.35 (K2), J501.36 (K3), R504.2
Other:
- moved on the sheet: R503
Changed lines of the file:
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@@
   (junction (at 209.55 86.36) (diameter 0) (color 0 0 0 0)
   )
-  (junction (at 168.91 52.07) (diameter 0) (color 0 0 0 0)
-  )
   (junction (at 120.65 90.17) (diameter 0) (color 0 0 0 0)
   )
@@
   )
   (junction (at 162.56 100.33) (diameter 0) (color 0 0 0 0)
-  )
-  (junction (at 179.07 41.91) (diameter 0) (color 0 0 0 0)
   )
   (junction (at 182.88 132.08) (diameter 0) (color 0 0 0 0)
@@
     (stroke (width 0) (type default) (color 0 0 0 0))
   )
-  (wire (pts (xy 168.91 41.91) (xy 179.07 41.91))
-    (stroke (width 0) (type default) (color 0 0 0 0))
-  )
   (wire (pts (xy 116.84 76.2) (xy 135.89 76.2))
     (stroke (width 0) (type default) (color 0 0 0 0))
@@
     (stroke (width 0) (type default) (color 0 0 0 0))
   )
-  (wire (pts (xy 179.07 41.91) (xy 187.96 41.91))
+  (wire (pts (xy 168.91 41.91) (xy 187.96 41.91))
     (stroke (width 0) (type default) (color 0 0 0 0))
   )
@@
     (stroke (width 0) (type default) (color 0 0 0 0))
   )
-  (wire (pts (xy 179.07 52.07) (xy 168.91 52.07))
-    (stroke (width 0) (type default) (color 0 0 0 0))
-  )
   (wire (pts (xy 120.65 86.36) (xy 120.65 90.17))
     (stroke (width 0) (type default) (color 0 0 0 0))
@@
     (stroke (width 0) (type default) (color 0 0 0 0))
   )
-  (wire (pts (xy 124.46 68.58) (xy 154.94 68.58))
+  (wire (pts (xy 124.46 68.58) (xy 152.4 68.58))
     (stroke (width 0) (type default) (color 0 0 0 0))
   )
@@
     (stroke (width 0) (type default) (color 0 0 0 0))
   )
-  (wire (pts (xy 179.07 50.8) (xy 179.07 52.07))
-    (stroke (width 0) (type default) (color 0 0 0 0))
-  )
   (wire (pts (xy 187.96 41.91) (xy 187.96 59.69))
     (stroke (width 0) (type default) (color 0 0 0 0))
@@
     (stroke (width 0) (type default) (color 0 0 0 0))
   )
-  (wire (pts (xy 162.56 68.58) (xy 167.64 68.58))
-    (stroke (width 0) (type default) (color 0 0 0 0))
-  )
-  (wire (pts (xy 179.07 41.91) (xy 179.07 43.18))
+  (wire (pts (xy 160.02 68.58) (xy 167.64 68.58))
     (stroke (width 0) (type default) (color 0 0 0 0))
   )
@@
   )
   (text "ILI9488 display (40pin FPC, 4-wire SPI interface)" (at 77.47 25.4 0)
+    (effects (font (size 1.27 1.27)) (justify left bottom))
+  )
+  (label "BL_K" (at 162.56 114.3 0)
+    (effects (font (size 1.27 1.27)) (justify left bottom))
+  )
+  (label "DIO_GND" (at 200.66 132.08 0)
     (effects (font (size 1.27 1.27)) (justify left bottom))
   )
@@
     )
   )
-  (symbol (lib_id "Device:C") (at 179.07 46.99 0) (unit 1)
-    (in_bom yes) (on_board yes)
-    (property "Reference" "C503" (id 0) (at 181.61 45.72 0)
-      (effects (font (size 1.27 1.27)) (justify left))
-    )
-    (property "Value" "100n" (id 1) (at 181.61 48.26 0)
-      (effects (font (size 1.27 1.27)) (justify left))
-    )
-    (property "Footprint" "Capacitor_SMD:C_0603_1608Metric" (id 2) (at 180.0352 50.8 0)
-      (effects (font (size 1.27 1.27)) hide)
-    )
-    (property "Datasheet" "~" (id 3) (at 179.07 46.99 0)
-      (effects (font (size 1.27 1.27)) hide)
-    )
-    (pin "1")
-    (pin "2")
-  )
   (symbol (lib_id "Device:R") (at 196.85 132.08 90) (unit 1)
     (in_bom yes) (on_board yes)
@@
     (pin "2")
   )
-  (symbol (lib_id "Device:R") (at 158.75 68.58 90) (unit 1)
-    (in_bom yes) (on_board yes)
-    (property "Reference" "R504" (id 0) (at 163.83 67.31 90))
-    (property "Value" "0" (id 1) (at 154.94 67.31 90))
-    (property "Footprint" "Resistor_SMD:R_0603_1608Metric" (id 2) (at 158.75 70.358 90)
-      (effects (font (size 1.27 1.27)) hide)
-    )
-    (property "Datasheet" "~" (id 3) (at 158.75 68.58 0)
+  (symbol (lib_id "Device:R") (at 156.21 68.58 90) (unit 1)
+    (in_bom yes) (on_board yes)
+    (property "Reference" "R503" (id 0) (at 161.29 67.31 90))
+    (property "Value" "0" (id 1) (at 152.4 67.31 90))
+    (property "Footprint" "Resistor_SMD:R_0603_1608Metric" (id 2) (at 156.21 70.358 90)
+      (effects (font (size 1.27 1.27)) hide)
+    )
+    (property "Datasheet" "~" (id 3) (at 156.21 68.58 0)
       (effects (font (size 1.27 1.27)) hide)
     )
@@
   (symbol (lib_id "Device:R") (at 156.21 119.38 90) (unit 1)
     (in_bom yes) (on_board yes)
-    (property "Reference" "R503" (id 0) (at 156.21 114.3 90))
+    (property "Reference" "R504" (id 0) (at 156.21 114.3 90))
     (property "Value" "5R6" (id 1) (at 156.21 116.84 90))
     (property "Footprint" "Resistor_SMD:R_0603_1608Metric" (id 2) (at 156.21 121.158 90)

Commit message: some mcu..
Connections:
- net CONN_SCL: now reaches J501.11 (SCL), R503.2
Other:
- moved on the sheet: R503
Changed lines of the file:
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@@
     (stroke (width 0) (type default) (color 0 0 0 0))
   )
-  (wire (pts (xy 124.46 68.58) (xy 152.4 68.58))
+  (wire (pts (xy 124.46 68.58) (xy 140.97 68.58))
     (stroke (width 0) (type default) (color 0 0 0 0))
   )
@@
     (stroke (width 0) (type default) (color 0 0 0 0))
   )
-  (wire (pts (xy 160.02 68.58) (xy 167.64 68.58))
+  (wire (pts (xy 148.59 68.58) (xy 167.64 68.58))
     (stroke (width 0) (type default) (color 0 0 0 0))
   )
@@
   )
   (label "BL_K" (at 162.56 114.3 0)
+    (effects (font (size 1.27 1.27)) (justify left bottom))
+  )
+  (label "CONN_SCL" (at 157.48 68.58 0)
     (effects (font (size 1.27 1.27)) (justify left bottom))
   )
@@
     (pin "2")
   )
-  (symbol (lib_id "Device:R") (at 156.21 68.58 90) (unit 1)
+  (symbol (lib_id "Device:R") (at 144.78 68.58 90) (unit 1)
     (in_bom yes) (on_board yes)
-    (property "Reference" "R503" (id 0) (at 161.29 67.31 90))
-    (property "Value" "0" (id 1) (at 152.4 67.31 90))
-    (property "Footprint" "Resistor_SMD:R_0603_1608Metric" (id 2) (at 156.21 70.358 90)
-      (effects (font (size 1.27 1.27)) hide)
-    )
-    (property "Datasheet" "~" (id 3) (at 156.21 68.58 0)
-      (effects (font (size 1.27 1.27)) hide)
-    )
+    (property "Reference" "R503" (id 0) (at 149.86 67.31 90))
+    (property "Value" "0" (id 1) (at 140.97 67.31 90))
+    (property "Footprint" "Resistor_SMD:R_0603_1608Metric" (id 2) (at 144.78 70.358 90)
+      (effects (font (size 1.27 1.27)) hide)
+    )
+    (property "Datasheet" "~" (id 3) (at 144.78 68.58 0)
+      (effects (font (size 1.27 1.27)) hide)
+    )
