File: grblPANEL_encoders.kicad_sch (KiCad schematic)
At the start: 20 parts, among them J701 Conn_01x04, J702 Conn_01x04, J703 Conn_01x04, J704 Conn_01x04

Commit message: Refresh
Parts:
- removed D702: D_TVS, symbol Device:D_TVS
- removed TP702: TestPoint, symbol Connector:TestPoint
- added D703: D_TVS, Diode_SMD:D_SOD-323, symbol Device:D_TVS
- added R701, R702, R703, R704, R705, R706, R707, R708: 200, Resistor_SMD:R_0603_1608Metric, symbol Device:R
- added TP703: TestPoint, Connector_Pin:Pin_D1.0mm_L10.0mm, symbol Connector:TestPoint
- D701, D704, D705, D706, D707, D708: footprint (none) -> Diode_SMD:D_SOD-323
- D702: renamed from D703; footprint (none) -> Diode_SMD:D_SOD-323
- J701, J702, J703, J704: footprint (none) -> TerminalBlock_4Ucon:TerminalBlock_4Ucon_1x04_P3.50mm_Horizontal
- TP701, TP704, TP705, TP706, TP707, TP708: footprint (none) -> Connector_Pin:Pin_D1.0mm_L10.0mm
- TP702: renamed from TP703; footprint (none) -> Connector_Pin:Pin_D1.0mm_L10.0mm
Connections:
- net +3V3: now also J701.3 (Pin_3), J702.3 (Pin_3), J703.3 (Pin_3), J704.3 (Pin_3); no longer J701.1 (Pin_1), J702.1 (Pin_1), J703.1 (Pin_1), J704.1 (Pin_1)
- net ENCODER_1_A: now also R701.1; no longer D702.2 (A2), J701.2 (Pin_2), TP701.1
- net ENCODER_1_B: now also R703.1; no longer D701.2 (A2), J701.3 (Pin_3), TP702.1
- net ENCODER_2_A: now also R702.1; no longer D707.2 (A2), J703.2 (Pin_2), TP705.1
- net ENCODER_2_B: now also R704.1; no longer D705.2 (A2), J703.3 (Pin_3), TP707.1
- net ENCODER_3_A: now also R705.1; no longer D704.2 (A2), J702.2 (Pin_2)
- net ENCODER_3_B: now also R707.1; no longer J702.3 (Pin_3), TP704.1
- net ENCODER_4_A: now also R706.1; no longer D708.2 (A2), J704.2 (Pin_2), TP706.1
- net ENCODER_4_B: now also R708.1; no longer D706.2 (A2), J704.3 (Pin_3), TP708.1
- net GND: now also D703.1 (A1)
- new net: D702.2 (A2), J701.2 (Pin_2), R703.2, TP702.1
- new net: D706.2 (A2), J703.2 (Pin_2), R707.2, TP706.1
- new net: D703.2 (A2), J702.1 (Pin_1), R702.2, TP703.1
- new net: D705.2 (A2), J703.1 (Pin_1), R705.2, TP705.1
- new net: D701.2 (A2), J701.1 (Pin_1), R701.2, TP701.1
- new net: D704.2 (A2), J702.2 (Pin_2), R704.2, TP704.1
- new net: D707.2 (A2), J704.1 (Pin_1), R706.2, TP707.1
- new net: D708.2 (A2), J704.2 (Pin_2), R708.2, TP708.1
Other:
- note added: "Note: Connector pinout to match rotary encoder breakouts @ https://github.com/dresco/RotaryEncoder"
- note removed: "Notes: Confirm connector pinout... Confirm connector footprint..."
- moved on the sheet: D701, D702, J701, TP701, TP702

Commit message: Status LED & annotation cleanup
Parts:
- renumbered D705 to D702, D702 to D703, D706 to D704, D703 to D705, D707 to D706, D704 to D707, J703 to J702, J702 to J703, R703 to R702, R705 to R703, R707 to R704, R702 to R705, R704 to R706, R706 to R707, TP705 to TP702, TP702 to TP703, TP706 to TP704, TP703 to TP705, TP707 to TP706, TP704 to TP707
Connections:
- net ENCODER_2_A: now also R703.1; no longer R705.1
- net ENCODER_2_B: now also R704.1; no longer R706.1
- net ENCODER_3_A: now also R705.1; no longer R703.1
- net ENCODER_3_B: now also R706.1; no longer R704.1
Changed lines of the file:
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@@
     (stroke (width 0) (type default) (color 0 0 0 0))
   )
-  (text "Quadrature encoder #2" (at 158.75 33.02 0)
+  (text "Quadrature encoder #3" (at 158.75 33.02 0)
     (effects (font (size 1.27 1.27)) (justify left bottom))
   )
-  (text "Quadrature encoder #3" (at 60.96 105.41 0)
+  (text "Quadrature encoder #2" (at 60.96 105.41 0)
     (effects (font (size 1.27 1.27)) (justify left bottom))
   )
@@
     (effects (font (size 1.27 1.27)) (justify left bottom))
   )
-  (global_label "ENCODER_2_A" (shape output) (at 185.42 52.07 180) (fields_autoplaced)
+  (global_label "ENCODER_3_A" (shape output) (at 185.42 52.07 180) (fields_autoplaced)
     (effects (font (size 1.27 1.27)) (justify right))
     (property "Intersheet References" "${INTERSHEET_REFS}" (id 0) (at 170.0045 51.9906 0)
@@
     )
   )
-  (global_label "ENCODER_3_A" (shape output) (at 87.63 124.46 180) (fields_autoplaced)
+  (global_label "ENCODER_2_A" (shape output) (at 87.63 124.46 180) (fields_autoplaced)
     (effects (font (size 1.27 1.27)) (justify right))
     (property "Intersheet References" "${INTERSHEET_REFS}" (id 0) (at 72.2145 124.3806 0)
@@
     )
   )
-  (global_label "ENCODER_3_B" (shape output) (at 87.63 127 180) (fields_autoplaced)
+  (global_label "ENCODER_2_B" (shape output) (at 87.63 127 180) (fields_autoplaced)
     (effects (font (size 1.27 1.27)) (justify right))
     (property "Intersheet References" "${INTERSHEET_REFS}" (id 0) (at 72.0331 126.9206 0)
@@
     )
   )
-  (global_label "ENCODER_2_B" (shape output) (at 185.42 54.61 180) (fields_autoplaced)
+  (global_label "ENCODER_3_B" (shape output) (at 185.42 54.61 180) (fields_autoplaced)
     (effects (font (size 1.27 1.27)) (justify right))
     (property "Intersheet References" "${INTERSHEET_REFS}" (id 0) (at 169.8231 54.5306 0)
@@
   (symbol (lib_id "Device:D_TVS") (at 111.76 66.04 90) (unit 1)
     (in_bom yes) (on_board yes)
-    (property "Reference" "D702" (id 0) (at 111.76 69.85 90)
+    (property "Reference" "D703" (id 0) (at 111.76 69.85 90)
       (effects (font (size 1.27 1.27)) (justify right))
     )
@@
   (symbol (lib_id "power:GND") (at 196.85 72.39 0) (unit 1)
     (in_bom yes) (on_board yes) (fields_autoplaced)
-    (property "Reference" "#PWR0704" (id 0) (at 196.85 78.74 0)
+    (property "Reference" "#PWR0707" (id 0) (at 196.85 78.74 0)
       (effects (font (size 1.27 1.27)) hide)
     )
@@
   (symbol (lib_id "Connector:TestPoint") (at 114.3 120.65 0) (unit 1)
     (in_bom yes) (on_board yes)
-    (property "Reference" "TP706" (id 0) (at 111.76 115.57 0)
+    (property "Reference" "TP704" (id 0) (at 111.76 115.57 0)
       (effects (font (size 1.27 1.27)) (justify left))
     )
@@
   (symbol (lib_id "Device:D_TVS") (at 203.2 66.04 90) (unit 1)
     (in_bom yes) (on_board yes)
-    (property "Reference" "D703" (id 0) (at 203.2 69.85 90)
+    (property "Reference" "D705" (id 0) (at 203.2 69.85 90)
       (effects (font (size 1.27 1.27)) (justify right))
     )
@@
   (symbol (lib_id "Connector_Generic:Conn_01x04") (at 121.92 127 0) (unit 1)
     (in_bom yes) (on_board yes)
-    (property "Reference" "J703" (id 0) (at 120.65 135.89 0)
+    (property "Reference" "J702" (id 0) (at 120.65 135.89 0)
       (effects (font (size 1.27 1.27)) (justify left))
     )
@@
   (symbol (lib_id "Connector:TestPoint") (at 114.3 48.26 0) (unit 1)
     (in_bom yes) (on_board yes)
-    (property "Reference" "TP702" (id 0) (at 111.76 43.18 0)
+    (property "Reference" "TP703" (id 0) (at 111.76 43.18 0)
       (effects (font (size 1.27 1.27)) (justify left))
     )
@@
   (symbol (lib_id "Device:R") (at 96.52 54.61 90) (unit 1)
     (in_bom yes) (on_board yes)
-    (property "Reference" "R703" (id 0) (at 101.6 53.34 90))
+    (property "Reference" "R702" (id 0) (at 101.6 53.34 90))
     (property "Value" "200" (id 1) (at 91.44 53.34 90))
     (property "Footprint" "Resistor_SMD:R_0603_1608Metric" (id 2) (at 96.52 56.388 90)
@@
   (symbol (lib_id "Connector:TestPoint") (at 205.74 48.26 0) (unit 1)
     (in_bom yes) (on_board yes)
-    (property "Reference" "TP703" (id 0) (at 201.93 43.18 0)
+    (property "Reference" "TP705" (id 0) (at 201.93 43.18 0)
       (effects (font (size 1.27 1.27)) (justify left))
     )
@@
   (symbol (lib_id "Connector:TestPoint") (at 107.95 120.65 0) (unit 1)
     (in_bom yes) (on_board yes)
-    (property "Reference" "TP705" (id 0) (at 104.14 115.57 0)
+    (property "Reference" "TP702" (id 0) (at 104.14 115.57 0)
       (effects (font (size 1.27 1.27)) (justify left))
     )
@@
   (symbol (lib_id "Device:D_TVS") (at 209.55 66.04 90) (unit 1)
     (in_bom yes) (on_board yes)
-    (property "Reference" "D704" (id 0) (at 209.55 69.85 90)
+    (property "Reference" "D707" (id 0) (at 209.55 69.85 90)
       (effects (font (size 1.27 1.27)) (justify right))
     )
@@
   (symbol (lib_id "Connector:TestPoint") (at 205.74 120.65 0) (unit 1)
     (in_bom yes) (on_board yes)
-    (property "Reference" "TP707" (id 0) (at 201.93 115.57 0)
+    (property "Reference" "TP706" (id 0) (at 201.93 115.57 0)
       (effects (font (size 1.27 1.27)) (justify left))
     )
@@
   (symbol (lib_id "Device:R") (at 194.31 54.61 90) (unit 1)
     (in_bom yes) (on_board yes)
-    (property "Reference" "R704" (id 0) (at 199.39 53.34 90))
+    (property "Reference" "R706" (id 0) (at 199.39 53.34 90))
     (property "Value" "200" (id 1) (at 189.23 53.34 90))
     (property "Footprint" "Resistor_SMD:R_0603_1608Metric" (id 2) (at 194.31 56.388 90)
@@
   (symbol (lib_id "Connector:TestPoint") (at 212.09 48.26 0) (unit 1)
     (in_bom yes) (on_board yes)
-    (property "Reference" "TP704" (id 0) (at 209.55 43.18 0)
+    (property "Reference" "TP707" (id 0) (at 209.55 43.18 0)
       (effects (font (size 1.27 1.27)) (justify left))
     )
@@
   (symbol (lib_id "Device:R") (at 96.52 127 90) (unit 1)
     (in_bom yes) (on_board yes)
-    (property "Reference" "R707" (id 0) (at 101.6 125.73 90))
+    (property "Reference" "R704" (id 0) (at 101.6 125.73 90))
     (property "Value" "200" (id 1) (at 91.44 125.73 90))
     (property "Footprint" "Resistor_SMD:R_0603_1608Metric" (id 2) (at 96.52 128.778 90)
@@
   (symbol (lib_id "Device:D_TVS") (at 203.2 138.43 90) (unit 1)
     (in_bom yes) (on_board yes)
-    (property "Reference" "D707" (id 0) (at 203.2 142.24 90)
+    (property "Reference" "D706" (id 0) (at 203.2 142.24 90)
       (effects (font (size 1.27 1.27)) (justify right))
     )
@@
   (symbol (lib_id "Device:R") (at 194.31 52.07 90) (unit 1)
     (in_bom yes) (on_board yes)
-    (property "Reference" "R702" (id 0) (at 199.39 50.8 90))
+    (property "Reference" "R705" (id 0) (at 199.39 50.8 90))
     (property "Value" "200" (id 1) (at 189.23 50.8 90))
     (property "Footprint" "Resistor_SMD:R_0603_1608Metric" (id 2) (at 194.31 53.848 90)
@@
   (symbol (lib_id "power:+3V3") (at 68.58 116.84 0) (unit 1)
     (in_bom yes) (on_board yes) (fields_autoplaced)
-    (property "Reference" "#PWR0705" (id 0) (at 68.58 120.65 0)
+    (property "Reference" "#PWR0702" (id 0) (at 68.58 120.65 0)
       (effects (font (size 1.27 1.27)) hide)
     )
@@
   (symbol (lib_id "Device:R") (at 96.52 124.46 90) (unit 1)
     (in_bom yes) (on_board yes)
-    (property "Reference" "R705" (id 0) (at 101.6 123.19 90))
+    (property "Reference" "R703" (id 0) (at 101.6 123.19 90))
     (property "Value" "200" (id 1) (at 91.44 123.19 90))
     (property "Footprint" "Resistor_SMD:R_0603_1608Metric" (id 2) (at 96.52 126.238 90)
@@
   (symbol (lib_id "power:GND") (at 99.06 144.78 0) (unit 1)
     (in_bom yes) (on_board yes) (fields_autoplaced)
-    (property "Reference" "#PWR0707" (id 0) (at 99.06 151.13 0)
+    (property "Reference" "#PWR0704" (id 0) (at 99.06 151.13 0)
       (effects (font (size 1.27 1.27)) hide)
     )
@@
   (symbol (lib_id "power:+3V3") (at 166.37 44.45 0) (unit 1)
     (in_bom yes) (on_board yes) (fields_autoplaced)
-    (property "Reference" "#PWR0702" (id 0) (at 166.37 48.26 0)
+    (property "Reference" "#PWR0705" (id 0) (at 166.37 48.26 0)
       (effects (font (size 1.27 1.27)) hide)
     )
@@
   (symbol (lib_id "Connector_Generic:Conn_01x04") (at 219.71 54.61 0) (unit 1)
     (in_bom yes) (on_board yes)
-    (property "Reference" "J702" (id 0) (at 218.44 63.5 0)
+    (property "Reference" "J703" (id 0) (at 218.44 63.5 0)
       (effects (font (size 1.27 1.27)) (justify left))
     )
@@
   (symbol (lib_id "Device:R") (at 194.31 124.46 90) (unit 1)
     (in_bom yes) (on_board yes)
-    (property "Reference" "R706" (id 0) (at 199.39 123.19 90))
+    (property "Reference" "R707" (id 0) (at 199.39 123.19 90))
     (property "Value" "200" (id 1) (at 189.23 123.19 90))
     (property "Footprint" "Resistor_SMD:R_0603_1608Metric" (id 2) (at 194.31 126.238 90)
@@
   (symbol (lib_id "Device:D_TVS") (at 105.41 138.43 90) (unit 1)
     (in_bom yes) (on_board yes)
-    (property "Reference" "D705" (id 0) (at 105.41 142.24 90)
+    (property "Reference" "D702" (id 0) (at 105.41 142.24 90)
       (effects (font (size 1.27 1.27)) (justify right))
     )
@@
   (symbol (lib_id "Device:D_TVS") (at 111.76 138.43 90) (unit 1)
     (in_bom yes) (on_board yes)
-    (property "Reference" "D706" (id 0) (at 111.76 142.24 90)
-      (effects (font (size 1.27 1.27)) (justify right))
-    )
+    (property "Reference" "D704" (id 0) (at 111.76 142.24 90)
+      (effects (font (size 1.27 1.27)) (justify right))
+    )

Commit message: PCB layout - WIP
Parts:
- J701, J702, J703, J704: footprint TerminalBlock_4Ucon:TerminalBlock_4Ucon_1x04_P3.50mm_Horizontal -> TerminalBlock_Phoenix:TerminalBlock_Phoenix_PT-1,5-4-3.5-H_1x04_P3.50mm_Horizontal
- TP701, TP702, TP703, TP704, TP705, TP706, TP707, TP708: footprint Connector_Pin:Pin_D1.0mm_L10.0mm -> TestPoint:TestPoint_THTPad_D2.0mm_Drill1.0mm
Connections:
- net ENCODER_1_A: now also TP701.1
- net ENCODER_1_B: now also TP703.1
- net ENCODER_2_A: now also TP702.1
- net ENCODER_2_B: now also TP704.1
- net ENCODER_3_A: now also TP705.1
- net ENCODER_3_B: now also TP707.1
- net ENCODER_4_A: now also TP706.1
- net ENCODER_4_B: now also TP708.1
- net CONN_ENC_1_B: now reaches D703.2 (A2), J701.2 (Pin_2), R702.2
- net CONN_ENC_1_B: no longer TP703.1
- net CONN_ENC_2_B: now reaches D704.2 (A2), J702.2 (Pin_2), R704.2
- net CONN_ENC_2_B: no longer TP704.1
- net CONN_ENC_3_A: now reaches D705.2 (A2), J703.1 (Pin_1), R705.2
- net CONN_ENC_3_A: no longer TP705.1
- net CONN_ENC_2_A: now reaches D702.2 (A2), J702.1 (Pin_1), R703.2
- net CONN_ENC_2_A: no longer TP702.1
- net CONN_ENC_1_A: now reaches D701.2 (A2), J701.1 (Pin_1), R701.2
- net CONN_ENC_1_A: no longer TP701.1
- net CONN_ENC_3_B: now reaches D707.2 (A2), J703.2 (Pin_2), R706.2
- net CONN_ENC_3_B: no longer TP707.1
- net CONN_ENC_4_A: now reaches D706.2 (A2), J704.1 (Pin_1), R707.2
- net CONN_ENC_4_A: no longer TP706.1
- net CONN_ENC_4_B: now reaches D708.2 (A2), J704.2 (Pin_2), R708.2
- net CONN_ENC_4_B: no longer TP708.1
Other:
- moved on the sheet: D701, D703, J701, R701, R702, TP701, TP703

Commit message: keypad test points
Parts:
- removed TP701, TP702, TP703, TP704, TP705, TP706, TP707, TP708: TestPoint, TestPoint:TestPoint_THTPad_D2.0mm_Drill1.0mm, symbol Connector:TestPoint
