File: grblPANEL_canbus.kicad_sch (KiCad schematic)
At the start: 14 parts, among them J301 Conn_01x02, U301 SN65HVD230

Commit message: canbus & modbus test points
Parts:
- removed TP303, TP304: TestPoint, TestPoint:TestPoint_THTPad_D2.0mm_Drill1.0mm, symbol Connector:TestPoint
Changed lines of the file:
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@@
   (junction (at 191.77 68.58) (diameter 0) (color 0 0 0 0)
   )
-  (junction (at 116.84 68.58) (diameter 0) (color 0 0 0 0)
-  )
-  (junction (at 121.92 71.12) (diameter 0) (color 0 0 0 0)
-  )
   (junction (at 209.55 68.58) (diameter 0) (color 0 0 0 0)
   )
@@
     (stroke (width 0) (type default) (color 0 0 0 0))
   )
-  (wire (pts (xy 121.92 62.23) (xy 121.92 71.12))
-    (stroke (width 0) (type default) (color 0 0 0 0))
-  )
   (polyline (pts (xy 199.39 91.44) (xy 185.42 91.44))
     (stroke (width 0) (type default) (color 0 0 0 0))
@@
     (stroke (width 0) (type default) (color 0 0 0 0))
   )
-  (wire (pts (xy 116.84 68.58) (xy 138.43 68.58))
-    (stroke (width 0) (type default) (color 0 0 0 0))
-  )
   (wire (pts (xy 62.23 62.23) (xy 62.23 66.04))
     (stroke (width 0) (type default) (color 0 0 0 0))
@@
     (stroke (width 0) (type default) (color 0 0 0 0))
   )
-  (wire (pts (xy 110.49 71.12) (xy 121.92 71.12))
+  (wire (pts (xy 110.49 71.12) (xy 161.29 71.12))
     (stroke (width 0) (type default) (color 0 0 0 0))
   )
@@
     (stroke (width 0) (type default) (color 0 0 0 0))
   )
-  (wire (pts (xy 116.84 62.23) (xy 116.84 68.58))
-    (stroke (width 0) (type default) (color 0 0 0 0))
-  )
   (wire (pts (xy 227.33 78.74) (xy 227.33 86.36))
     (stroke (width 0) (type default) (color 0 0 0 0))
@@
     (stroke (width 0) (type default) (color 0 0 0 0))
   )
-  (wire (pts (xy 121.92 71.12) (xy 161.29 71.12))
-    (stroke (width 0) (type default) (color 0 0 0 0))
-  )
   (wire (pts (xy 100.33 78.74) (xy 100.33 86.36))
     (stroke (width 0) (type default) (color 0 0 0 0))
@@
     (stroke (width 0) (type default) (color 0 0 0 0))
   )
-  (wire (pts (xy 110.49 68.58) (xy 116.84 68.58))
+  (wire (pts (xy 110.49 68.58) (xy 138.43 68.58))
     (stroke (width 0) (type default) (color 0 0 0 0))
   )
@@
     (pin "2")
   )
-  (symbol (lib_id "Connector:TestPoint") (at 116.84 62.23 0) (unit 1)
-    (in_bom yes) (on_board yes)
-    (property "Reference" "TP303" (id 0) (at 113.03 57.15 0)
-      (effects (font (size 1.27 1.27)) (justify left))
-    )
-    (property "Value" "TestPoint" (id 1) (at 119.38 60.1979 0)
-      (effects (font (size 1.27 1.27)) (justify left) hide)
-    )
-    (property "Footprint" "TestPoint:TestPoint_THTPad_D2.0mm_Drill1.0mm" (id 2) (at 121.92 62.23 0)
-      (effects (font (size 1.27 1.27)) hide)
-    )
-    (property "Datasheet" "~" (id 3) (at 121.92 62.23 0)
-      (effects (font (size 1.27 1.27)) hide)
-    )
-    (pin "1")
-  )
   (symbol (lib_id "Connector:TestPoint") (at 62.23 62.23 0) (unit 1)
     (in_bom yes) (on_board yes)
@@
     (pin "2")
   )
-  (symbol (lib_id "Connector:TestPoint") (at 121.92 62.23 0) (unit 1)
-    (in_bom yes) (on_board yes)
-    (property "Reference" "TP304" (id 0) (at 120.65 57.15 0)
-      (effects (font (size 1.27 1.27)) (justify left))
-    )
-    (property "Value" "TestPoint" (id 1) (at 124.46 60.1979 0)
-      (effects (font (size 1.27 1.27)) (justify left) hide)
-    )
-    (property "Footprint" "TestPoint:TestPoint_THTPad_D2.0mm_Drill1.0mm" (id 2) (at 127 62.23 0)
-      (effects (font (size 1.27 1.27)) hide)
-    )
-    (property "Datasheet" "~" (id 3) (at 127 62.23 0)
-      (effects (font (size 1.27 1.27)) hide)
-    )
-    (pin "1")
-  )
   (symbol (lib_id "Interface_CAN_LIN:SN65HVD230") (at 100.33 68.58 0) (unit 1)

Commit message: Place and route changes from schematic
Headers for serial console.
DNP components to v7 format.
Power status components.
LEDs to bottom side, plus silkscreen.
Parts:
- C302, C303, R301: now not fitted
Changed lines of the file:
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@@
   )
   (symbol (lib_id "Device:C") (at 191.77 82.55 0) (unit 1)
-    (in_bom yes) (on_board yes) (dnp no)
+    (in_bom yes) (on_board yes) (dnp yes)
     (property "Reference" "C303" (at 193.04 80.01 0)
       (effects (font (size 1.27 1.27)) (justify left))
@@
   )
   (symbol (lib_id "Device:C") (at 191.77 72.39 0) (unit 1)
-    (in_bom yes) (on_board yes) (dnp no)
+    (in_bom yes) (on_board yes) (dnp yes)
     (property "Reference" "C302" (at 193.04 69.85 0)
       (effects (font (size 1.27 1.27)) (justify left))
@@
   )
   (symbol (lib_id "Device:R") (at 74.93 80.01 0) (unit 1)
-    (in_bom yes) (on_board yes) (dnp no)
+    (in_bom yes) (on_board yes) (dnp yes)
     (property "Reference" "R301" (at 76.2 78.74 0)
       (effects (font (size 1.27 1.27)) (justify left))
