File: grblPANEL_mcu.kicad_sch (KiCad schematic)
At the start: 33 parts, among them J201 2x5x1.27mm, J202 USB_C_Receptacle_USB2.0, SW201 SW_Push, SW202 SW_Push, U201 STM32G0B1CxTxN, U202 USBLC6-2SC6, Y201 8MHz

Commit message: Board changes for Rev B
Import changes from schematic.

Place and route changes from schematic:
Headers for serial console.
DNP components to v7 format.
Power status components.
LEDs to bottom side, plus silkscreen.

Update schematic page settings (RevB).

Update PCB page settings (RevB).

Silkscreen & test point tweaks.
Parts:
- D201: footprint LED_SMD:LED_1206_3216Metric_ReverseMount_Hole1.8x2.4mm -> LED_SMD:LED_0603_1608Metric
Changed lines of the file:
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@@
   (title_block
     (title "grblPANEL")
-    (date "2022-12-12")
-    (rev "0.1")
+    (date "2023-03-09")
+    (rev "B")
     (company "dresco")
   )
@@
       (effects (font (size 1.27 1.27)) (justify right))
     )
-    (property "Footprint" "LED_SMD:LED_1206_3216Metric_ReverseMount_Hole1.8x2.4mm" (at 135.89 55.88 0)
-      (effects (font (size 1.27 1.27)) hide)
-    )
+    (property "Footprint" "LED_SMD:LED_0603_1608Metric" (at 135.89 55.88 0)
+      (effects (font (size 1.27 1.27)) hide)
+    )

Commit message: Green LED resistor changes
Reduce the intensity of the green status LEDs, resistors changed
from 1k to 4k7
Parts:
- R205: value 1k -> 4k7
Changed lines of the file:
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@@
       (effects (font (size 1.27 1.27)))
     )
-    (property "Value" "1k" (at 128.27 58.42 90)
+    (property "Value" "4k7" (at 128.27 58.42 90)
       (effects (font (size 1.27 1.27)))
     )
