File: grblPANEL_power.kicad_sch (KiCad schematic)
At the start: 29 parts, among them J101 Conn_01x02, U101 TL431, U102 MAX17612A, U103 AZ1117-3.3

Commit message: Board changes for Rev B
Import changes from schematic.

Place and route changes from schematic:
Headers for serial console.
DNP components to v7 format.
Power status components.
LEDs to bottom side, plus silkscreen.

Update schematic page settings (RevB).

Update PCB page settings (RevB).

Silkscreen & test point tweaks.
Parts:
- added R109, R110: 680, Resistor_SMD:R_0603_1608Metric, symbol Device:R
- D103, D104, D106: footprint LED_SMD:LED_1206_3216Metric_ReverseMount_Hole1.8x2.4mm -> LED_SMD:LED_0603_1608Metric
- R101: value 5k6 -> 4k7
- R103: renamed from R105; now not fitted
- R112: renamed from R110; now not fitted
- renumbered R104 to R102, R102 to R104, R103 to R105, R109 to R111, R111 to R113, R112 to R114
Connections:
- net FLAG: now also R109.2; no longer D103.1 (K)
- net UVOV: now also R110.2; no longer D104.1 (K)
- new net: D104.1 (K), R110.1
- new net: D103.1 (K), R109.1
Other:
- note added: "FLAG and UVOV status pins are open drain, max voltage ~6v Shunt regulator to generate ~2.5v LED supply from unprotected input Vin resistor sized for ~2mA @ 12v (9.5v drop), LED resistor sized for ~1mA (0.7v drop), leaving ~1mA to maintain regulation when lit"
- note added: "todo: power leds - confirm suitable resistor values after testing - make a simple test board at the same time.."
- note removed: "FLAG and UVOV status pins are open drain, max voltage ~6v Shunt regulator to generate ~2.5v LED supply from unprotected input Resistor sized for ~2mA @ 12v"
- note removed: "todo: power leds - confirm suitable resistor & capacitor values after testing"
- moved on the sheet: D101, D103, D104, R101, R102, U101

Commit message: Green LED resistor changes
Reduce the intensity of the green status LEDs, resistors changed
from 1k to 4k7
Parts:
- R114: value 1k -> 4k7
Changed lines of the file:
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@@
   (symbol (lib_id "Device:R") (at 248.92 90.17 0) (unit 1)
     (in_bom yes) (on_board yes) (dnp no) (fields_autoplaced)
-    (property "Reference" "R114" (at 251.46 88.8999 0)
+    (property "Reference" "R114" (at 251.46 89.535 0)
       (effects (font (size 1.27 1.27)) (justify left))
     )
-    (property "Value" "1k" (at 251.46 91.4399 0)
+    (property "Value" "4k7" (at 251.46 92.075 0)
       (effects (font (size 1.27 1.27)) (justify left))
     )
